File: buffer.sch (KiCad schematic (older format))
At the start: 32 parts, among them J10 Drive+, J11 Sense-, J12 Drive-, J9 Sense+, Q4 Q_NPN_BCE, Q5 Q_PNP_BCE, U1 ADA4523-1, U2 ADA4523-1

Commit message: srdgv
Connections:
- net at Q5.2 (C): now also C31.1, C32.1, R935.2; no longer R933.1
- new net: Q5.3 (E), R933.1
Changed lines of the file:
@@
 F 3 "https://www.mouser.de/datasheet/2/115/FZT751Q-1532260.pdf" H 6500 4850 50  0001 C CNN
 	1    6500 4850
-	1    0    0    -1
+	1    0    0    1
 $EndComp
 $Comp
