File: ltz10v.kicad_pcb (KiCad board)
At the start: 4 copper layers, 108 x 57 mm, 1012 parts, among them J1 Conn_01x04, J10 Drive+, J11 Sense-, J12 Drive-, J2 Conn_01x04, J3 AC1, J4 Conn_01x04, J5 Conn_01x04, J6 Bat-, J7 Bat+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

Commit message: srdgv
Parts:
- moved C32 68.1 mm to (153.5, 103.5), turned to 180 degrees
- moved R939 67.5 mm to (143.0, 89.0), turned to 90 degrees
- moved C31 66.8 mm to (153.5, 101.0), turned to 180 degrees
- moved R938 65.1 mm to (163.5, 101.5), turned to 180 degrees
- moved J11 64.6 mm to (136.5, 67.5)
- moved RN1 57.5 mm to (162.0, 98.0)
- moved U2 56.0 mm to (166.0, 90.5), turned to 180 degrees
- moved R935 55.9 mm to (153.5, 98.5)
- moved U1 54.3 mm to (166.0, 81.5), turned to 180 degrees
- moved R942 53.7 mm to (172.0, 92.0)
- moved C29 53.6 mm to (166.0, 94.5)
- moved R933 52.3 mm to (146.5, 91.5), turned to 180 degrees
- moved R934 51.7 mm to (160.1, 91.0)
- moved R940 50.0 mm to (172.0, 99.0)
- moved R932 49.4 mm to (146.5, 87.0)
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Routing:
- net Net-(C29-Pad2): track 0.00 -> 105.5 mm
- net GND: track 169.4 -> 227.2 mm, vias 26 -> 29
- net /buffer/Zener_drive+: track 0.00 -> 57.1 mm
- net Net-(J9-Pad1): track 0.00 -> 56.8 mm
- net +12V: track 69.7 -> 109.5 mm, vias 6 -> 8
- net Net-(C28-Pad2): track 0.00 -> 34.5 mm
- net /buffer/Zener_drive-: track 0.00 -> 31.5 mm
- net Net-(R938-Pad2): track 0.00 -> 28.7 mm
- net Net-(J12-Pad1): track 0.00 -> 26.3 mm
- net Net-(J10-Pad1): track 0.00 -> 23.7 mm
- net Net-(C26-Pad2): track 0.00 -> 17.2 mm
- net Net-(R942-Pad1): track 0.00 -> 12.7 mm
- net Net-(Q5-Pad2): track 0.00 -> 10.0 mm
- net Net-(Q4-Pad3): track 0.00 -> 9.30 mm
- net Net-(C31-Pad1): track 0.00 -> 8.62 mm
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
Commit message: added fab outputs
Other:
- board text added: "KX 10V Buffer"
- board text added: "reps Nov 2020"
